File: PCB/flypi_pcb_kicad/flypi.sch (KiCad schematic (older format))
At the start: 39 parts, among them CON1 BARREL_JACK, J12 USB_A, P1 PeltS1S2, P10 RGB RG-B, P3 Fan+-, P4 Therm +s-, P5 HP1+-, P6 HP2+-, P7 servo +s-, P8 Ring +-s, P9 I2C +-scsd, Q1 1A_NPN_EBC, Q2 1A-NPN-EBC, Q3 1A_NPN_EBC, Q4 1A_NPN_EBC, U1 LM2596, U2 LM2596, U4 L298N, U5 arduino_mini

Commit message: Revert "Prepare for kitspace (#22)"
This reverts commit 9aa00d109e1364754c2a30ef1fc76aca93cc7955.
Parts:
- removed J12: USB_A, Connectors:USB_A_Vertical, symbol USB_A
- added C3: 680µ, Capacitors_ThroughHole:C_Radial_D10_L21_P5, symbol CP1
- added C4: 220µ, Capacitors_ThroughHole:C_Radial_D8_L13_P3.8, symbol CP1
- added D2: Schottky 5A, Diodes_ThroughHole:Diode_DO-201AD_Horizontal_RM15, symbol D_Schottky
- added L3: 33µH, Inductors_NEOSID:Neosid_Inductor_MA-Bs75, symbol INDUCTOR
- added P2: Pi+-, Terminal_Blocks:TerminalBlock_Pheonix_PT-3.5mm_2pol, symbol CONN_01X02
- added U3: LM2596, footprints:LM2596, symbol LM2596
- 1k1, R2, R3, R4, R5, R7, R8, R9: footprint Resistors_THT:R_Box_L13.0mm_W4.0mm_P9.00mm -> Resistors_ThroughHole:Resistor_Horizontal_RM10mm
- C8: value 100n -> 0.1µ
- P1, P3, P5, P6: footprint Connectors_JST:JST_EH_S02B-EH_02x2.50mm_Angled -> Terminal_Blocks:TerminalBlock_Pheonix_PT-3.5mm_2pol; symbol Conn_01x02 -> CONN_01X02
- P10: footprint Connectors_JST:JST_EH_S04B-EH_04x2.50mm_Angled -> Terminal_Blocks:TerminalBlock_Pheonix_PT-3.5mm_4pol; symbol Conn_01x04 -> CONN_01X04
- P4, P7, P8: footprint Connectors_JST:JST_EH_S03B-EH_03x2.50mm_Angled -> Terminal_Blocks:TerminalBlock_Pheonix_PT-3.5mm_3pol; symbol Conn_01x03 -> CONN_01X03
- P9: value I2C +-scsd -> matrix +-scsd; footprint Socket_Strips:Socket_Strip_Straight_1x04_Pitch2.54mm -> Terminal_Blocks:TerminalBlock_Pheonix_PT-3.5mm_4pol; symbol Conn_01x04 -> CONN_01X04
- Q1, Q3, Q4: value 1A_NPN_EBC -> 1A_NPN_ECB; footprint TO_SOT_Packages_THT:TO-92_Inline_Wide -> TO_SOT_Packages_THT:TO-92_Inline_Narrow_Oval; symbol 2N2219 -> Q_NPN_ECB
- Q2: value 1A-NPN-EBC -> 1A-NPN-ECB; footprint TO_SOT_Packages_THT:TO-92_Inline_Wide -> TO_SOT_Packages_THT:TO-92_Inline_Narrow_Oval; symbol 2N2219 -> Q_NPN_ECB
- R1: value 20W -> 1 - 18W; footprint TO_SOT_Packages_THT:TO-220-2_Vertical -> footprints:high_load_res; symbol R -> HighLoadRes
- U5: footprint arduino_nano:DIP-30_W15.24mm_LongPads -> Housings_DIP:DIP-32_W15.24mm_LongPads
Connections:
- net GND: now also R1.1, C3.2, C4.2, D2.2 (A), P2.2 (P2), U3.3 (Ground), U3.5 (On/Off); no longer R1.2
- net at C1.1, C10.2, C2.1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: now also Q1.2 (C), C3.1, U3.1 (Power_in); no longer Q1.3 (C)
- net at C6.1, L2.2, U1.4 (Feedback): now also P2.1 (P1)
- net at Q2.2 (C): now also Q3.2 (C), Q4.2 (C), C4.1, L3.2, U3.4 (Feedback); no longer R2.1
- net at C5.1, L1.2, P8.1 (P1)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: no longer Q2.3 (C), Q3.3 (C), Q4.3 (C)
- net at R4.1: now also Q3.3 (B); no longer Q3.2 (B)
- net at R5.1: now also Q4.3 (B); no longer Q4.2 (B)
- net at U4.1 (Current_sensing_A): now also R1.2; no longer R1.1
- net at U4.2 (Output1): now also P1.1 (P1); no longer P1.2 (Pin_2)
- net at U4.3 (Output2): now also P1.2 (P2); no longer P1.1 (Pin_1)
- net at R3.1: now also Q1.3 (B); no longer Q1.2 (B)
- new net: D2.1 (K), L3.1, U3.2 (Power_out)
- new net: Q2.3 (B), R2.1
- no-connect marks 20 -> 19

Commit message: Prepare for kitspace (#22)
* update to pcbs. Both SMD and new through hole. PCB is untested.

* update 3d print files, and start the idea of having a library for common structures in the pieces

* change to gerber files

* update to pcb labels (corrected inverted values)

* removed matrix commands from Arduino

* major revision to python code. Reduced the number of recursive functions and data transmitted to arduino are now done only via flypiapp.py. Seems to have fixed protocols bugs and speeded up the Peltier temperature display

* cleaned up arduino code. Changed answer token and removed code related to matrix and unused ring functions

* created individual files for each part to be 3D printed. Should make life easier for creating new parts and placing parts to be printed in batches. As well as rounding edges

* updated the PCB. Removed one of the voltage regulators (as everything seem to work fine with just 2. Changed the plugs so that the cables cab be bought crimmped.)

* 3D print files cleanup

* updated pcb, so that screw holes are equidistant from board edges

* moved untested scads to a specific folder and restored the already tested files

* Update README.md

* Update README.md

* commented out libraries necessary for matrix

* update arduino code for ring with 4 leds per bit

* Start a kitspace BOM for the SMD version

* Add kitspace.yaml

* update gerber1 folder to gerber

* Update kitspace.yaml

changed the folder where kitspace will look for pcb and gerber

* move gerber zip

* update gebers

* found bug in gerbers
Parts:
- removed C3: 680µ, Capacitors_ThroughHole:C_Radial_D10_L21_P5, symbol CP1
- removed C4: 220µ, Capacitors_ThroughHole:C_Radial_D8_L13_P3.8, symbol CP1
- removed D2: Schottky 5A, Diodes_ThroughHole:Diode_DO-201AD_Horizontal_RM15, symbol D_Schottky
- removed L3: 33µH, Inductors_NEOSID:Neosid_Inductor_MA-Bs75, symbol INDUCTOR
- removed P2: Pi+-, Terminal_Blocks:TerminalBlock_Pheonix_PT-3.5mm_2pol, symbol CONN_01X02
- removed U3: LM2596, footprints:LM2596, symbol LM2596
- added J12: USB_A, Connectors:USB_A_Vertical, symbol USB_A
- 1k1, R2, R3, R4, R5, R7, R8, R9: footprint Resistors_ThroughHole:Resistor_Horizontal_RM10mm -> Resistors_THT:R_Box_L13.0mm_W4.0mm_P9.00mm
- C8: value 0.1µ -> 100n
- P1, P3, P5, P6: footprint Terminal_Blocks:TerminalBlock_Pheonix_PT-3.5mm_2pol -> Connectors_JST:JST_EH_S02B-EH_02x2.50mm_Angled; symbol CONN_01X02 -> Conn_01x02
- P10: footprint Terminal_Blocks:TerminalBlock_Pheonix_PT-3.5mm_4pol -> Connectors_JST:JST_EH_S04B-EH_04x2.50mm_Angled; symbol CONN_01X04 -> Conn_01x04
- P4, P7, P8: footprint Terminal_Blocks:TerminalBlock_Pheonix_PT-3.5mm_3pol -> Connectors_JST:JST_EH_S03B-EH_03x2.50mm_Angled; symbol CONN_01X03 -> Conn_01x03
- P9: value matrix +-scsd -> I2C +-scsd; footprint Terminal_Blocks:TerminalBlock_Pheonix_PT-3.5mm_4pol -> Socket_Strips:Socket_Strip_Straight_1x04_Pitch2.54mm; symbol CONN_01X04 -> Conn_01x04
- Q1, Q3, Q4: value 1A_NPN_ECB -> 1A_NPN_EBC; footprint TO_SOT_Packages_THT:TO-92_Inline_Narrow_Oval -> TO_SOT_Packages_THT:TO-92_Inline_Wide; symbol Q_NPN_ECB -> 2N2219
- Q2: value 1A-NPN-ECB -> 1A-NPN-EBC; footprint TO_SOT_Packages_THT:TO-92_Inline_Narrow_Oval -> TO_SOT_Packages_THT:TO-92_Inline_Wide; symbol Q_NPN_ECB -> 2N2219
- R1: value 1 - 18W -> 20W; footprint footprints:high_load_res -> TO_SOT_Packages_THT:TO-220-2_Vertical; symbol HighLoadRes -> R
- U5: footprint Housings_DIP:DIP-32_W15.24mm_LongPads -> arduino_nano:DIP-30_W15.24mm_LongPads
Connections:
- net GND: now also R1.2, J12.4 (GND), J12.5 (Shield); no longer R1.1
- net at C1.1, C10.2, C2.1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: now also Q1.3 (C); no longer Q1.2 (C)
- net at C6.1, L2.2, U1.4 (Feedback): now also J12.1 (VBUS)
- net at R2.1: now also Q2.2 (B); no longer Q2.3 (B)
- net at Q3.3 (C): now also C5.1, L1.2, P8.1 (Pin_1), P9.1 (Pin_1), Q2.3 (C), Q4.3 (C), U2.4 (Feedback); no longer R4.1
- net at R5.1: now also Q4.2 (B); no longer Q4.3 (B)
- net at U4.1 (Current_sensing_A): now also R1.1; no longer R1.2
- net at U4.2 (Output1): now also P1.2 (Pin_2); no longer P1.1 (P1)
- net at U4.3 (Output2): now also P1.1 (Pin_1); no longer P1.2 (P2)
- net at R3.1: now also Q1.2 (B); no longer Q1.3 (B)
- new net: Q3.2 (B), R4.1
- no-connect marks 19 -> 20
